File: PCB/BoardKeys.kicad_sch (KiCad schematic)
At the start: 140 parts, among them SW1 SW_Push, SW10 SW_Push, SW2 SW_Push, SW3 SW_Push, SW4 SW_Push, SW5 SW_Push, SW6 SW_Push, SW7 SW_Push, SW8 SW_Push, SW9 SW_Push

Commit message: Placed all switches on main PCB
Parts:
- removed STABSPACEL1: MX_stab, PCM_marbastlib-mx:STAB_MX_2.25u, symbol PCM_marbastlib-mx:MX_stab
- added STABLSHIFT1: MX_stab, PCM_marbastlib-mx:STAB_MX_2.25u, symbol PCM_marbastlib-mx:MX_stab
- STABBACK1: footprint PCM_marbastlib-mx:STAB_MX_2.25u -> PCM_marbastlib-mx:STAB_MX_2u
- STABSPACE1: renamed from STABSPACER1; footprint PCM_marbastlib-mx:STAB_MX_2.25u -> PCM_marbastlib-mx:STAB_MX_6.25u
- renumbered SW10 to SW0
Other:
- moved on the sheet: STABSPACE1
