File: PCB/65ROL-PCB.kicad_pcb (KiCad board)
At the start: 2 copper layers, 141 parts, among them SW0 SW_Push, SW1 SW_Push, SW2 SW_Push, SW3 SW_Push, SW4 SW_Push, SW5 SW_Push, SW6 SW_Push, SW7 SW_Push, SW8 SW_Push, SW9 SW_Push

Commit message: Placed all diodes and made edge
Parts:
- D'1, D,1, D-1, D.1, D/1, D1, D10, D2, D3, D4, D5, D6, D7, D8, D9, D;1, D=1, DA1, DB1, DBACK1, DC1, DCAPS1, DD1, DDEL1, DDOWN1, DE1, DENTER1, DESC1, DF1, DG1, DH1, DI1, DINS1, DJ1, DK1, DL1, DLALT1, DLCTRL1, DLEFT1, DLSHIFT1, DLWIN1, DM1, DN1, DO1, DP1, DPDN1, DPUP1, DQ1, DR1, DRALT1, DRCTRL1, DRIGHT1, DRSHIFT1, DRWIN1, DS1, DSPACE1, DT1, DTAB1, DU1, DUP1, DV1, DW1, DX1, DY1, DZ1, D[1, D\1, D]1: moved to B.Cu
- moved DPUP1 402.1 mm to (329.8, -40.2), turned to 90 degrees
- moved DRIGHT1 399.0 mm to (329.8, 1.40), turned to 90 degrees
- moved DPDN1 399.0 mm to (329.8, -19.4), turned to 90 degrees
- moved DDEL1 383.9 mm to (329.8, -81.8), turned to 90 degrees
- moved D\1 376.5 mm to (304.8, -61.0), turned to 90 degrees
- moved DUP1 367.6 mm to (309.0, -19.4), turned to 90 degrees
- moved DINS1 363.2 mm to (329.8, -61.0), turned to 90 degrees
- moved DBACK1 359.8 mm to (309.0, -81.8), turned to 90 degrees
- moved DENTER1 355.2 mm to (309.0, -40.2), turned to 90 degrees
- moved D]1 353.7 mm to (279.8, -61.0), turned to 90 degrees
- moved DRSHIFT1 353.6 mm to (280.4, -19.6), turned to 90 degrees
- moved DDOWN1 346.2 mm to (309.0, 1.41), turned to 90 degrees
- moved DRCTRL1 336.6 mm to (267.4, 1.41), turned to 90 degrees
- moved D[1 331.7 mm to (259.0, -61.0), turned to 90 degrees
- moved D-1 321.9 mm to (248.6, -81.8), turned to 90 degrees
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Connections:
- A2 pad 20: /Board Keys/ROW0 -> unconnected-(A2-GPIO15-Pad20)
- A2 pad 21: /R1 -> /R0
- A2 pad 22: /R2 -> /R1
- A2 pad 24: /R3 -> /R2
- A2 pad 25: /R4 -> /R3
- A2 pad 26: unconnected-(A2-GPIO20-Pad26) -> /R4
- D-1 pad 1: /Board Keys/ROW0 -> /R0
- D1 pad 1: /Board Keys/ROW0 -> /R0
- D10 pad 1: /Board Keys/ROW0 -> /R0
- D2 pad 1: /Board Keys/ROW0 -> /R0
- D3 pad 1: /Board Keys/ROW0 -> /R0
- D4 pad 1: /Board Keys/ROW0 -> /R0
- D5 pad 1: /Board Keys/ROW0 -> /R0
- D6 pad 1: /Board Keys/ROW0 -> /R0
- D7 pad 1: /Board Keys/ROW0 -> /R0
- D8 pad 1: /Board Keys/ROW0 -> /R0
- D9 pad 1: /Board Keys/ROW0 -> /R0
- D=1 pad 1: /Board Keys/ROW0 -> /R0
- DBACK1 pad 1: /Board Keys/ROW0 -> /R0
- DDEL1 pad 1: /Board Keys/ROW0 -> /R0
- DESC1 pad 1: /Board Keys/ROW0 -> /R0
Routing:
- net /Board Keys/COL14: track 0.00 -> 361.3 mm
- net /Board Keys/COL12: track 0.00 -> 325.4 mm
- net /Board Keys/COL11: track 0.00 -> 304.2 mm
- net /Board Keys/COL10: track 0.00 -> 285.9 mm
- net /Board Keys/COL13: track 0.00 -> 275.4 mm
- net /Board Keys/COL9: track 0.00 -> 270.2 mm
- net /Board Keys/COL8: track 0.00 -> 252.0 mm
- net /Board Keys/COL7: track 0.00 -> 206.1 mm
- net /Board Keys/COL5: track 0.00 -> 196.2 mm
- net /Board Keys/COL6: track 0.00 -> 187.9 mm
- net /Board Keys/COL4: track 0.00 -> 153.9 mm
- net /Board Keys/COL2: track 0.00 -> 143.8 mm
- net /Board Keys/COL3: track 0.00 -> 135.6 mm
- net /Board Keys/COL1: track 0.00 -> 130.3 mm
- net /Board Keys/COL0: track 0.00 -> 108.3 mm
Other:
- board outline added: 334.2 x 133.2 mm

Commit message: Routed keyboard and made ground fill
Parts:
- moved A2 150.7 mm to (-7.54, 45.5)
- moved D,1 150.7 mm to (203.1, 131.0)
- moved D-1 150.7 mm to (241.7, 68.8)
- moved D.1 150.7 mm to (223.9, 131.0)
- moved D/1 150.7 mm to (244.7, 131.0)
- moved D2 150.7 mm to (54.5, 68.8)
- moved D4 150.7 mm to (96.1, 68.8)
- moved D5 150.7 mm to (116.9, 68.8)
- moved D6 150.7 mm to (137.7, 68.8)
- moved D7 150.7 mm to (158.5, 68.8)
- moved D8 150.7 mm to (179.3, 68.8)
- moved D9 150.7 mm to (200.1, 68.8)
- moved DA1 150.7 mm to (49.5, 110.4)
- moved DB1 150.7 mm to (140.7, 131.0)
- moved DC1 150.7 mm to (99.1, 131.0)
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Routing:
- net /R4: track 0.00 -> 465.3 mm
- net /R3: track 0.00 -> 421.5 mm
- net /R2: track 0.00 -> 412.4 mm
- net /R1: track 0.00 -> 389.2 mm
- net /R0: track 0.00 -> 374.8 mm
- net Net-(DLSHIFT1-A): track 0.00 -> 22.2 mm
- net Net-(DENTER1-A): track 0.00 -> 22.1 mm
- net Net-(DBACK1-A): track 0.00 -> 19.7 mm
- net Net-(DRSHIFT1-A): track 0.00 -> 10.4 mm
- net Net-(DCAPS1-A): track 0.00 -> 10.4 mm
- net Net-(DTAB1-A): track 0.00 -> 10.4 mm
- net Net-(DESC1-A): track 0.00 -> 10.3 mm
- net Net-(DY1-A): track 0.00 -> 10.3 mm
- net Net-(D'1-A): track 0.00 -> 10.3 mm
- net Net-(DUP1-A): track 0.00 -> 10.3 mm
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- added copper zone on B.Cu, net GND
- added copper zone on F.Cu, net GND
Other:
- board size 334.2 x 133.2 mm -> 333.8 x 133.2 mm

Commit message: Added LEDs to schematic and PCB
Parts:
- added LED'1: SK6812MINI-E, HackClubCarePackage:SK6812MINI-E_fixed, F.Cu at (238.4, 97.1)
- added LED,1: SK6812MINI-E, HackClubCarePackage:SK6812MINI-E_fixed, F.Cu at (184.0, 117.9)
- added LED-1: SK6812MINI-E, HackClubCarePackage:SK6812MINI-E_fixed, F.Cu at (222.6, 55.5)
- added LED.1: SK6812MINI-E, HackClubCarePackage:SK6812MINI-E_fixed, F.Cu at (204.8, 117.9)
- added LED/1: SK6812MINI-E, HackClubCarePackage:SK6812MINI-E_fixed, F.Cu at (225.6, 117.9)
- added LED0: SK6812MINI-E, HackClubCarePackage:SK6812MINI-E_fixed, F.Cu at (201.8, 55.5)
- added LED1: SK6812MINI-E, HackClubCarePackage:SK6812MINI-E_fixed, F.Cu at (14.6, 55.5)
- added LED2: SK6812MINI-E, HackClubCarePackage:SK6812MINI-E_fixed, F.Cu at (35.4, 55.5)
- added LED3: SK6812MINI-E, HackClubCarePackage:SK6812MINI-E_fixed, F.Cu at (56.2, 55.5)
- added LED4: SK6812MINI-E, HackClubCarePackage:SK6812MINI-E_fixed, F.Cu at (77.0, 55.5)
- added LED5: SK6812MINI-E, HackClubCarePackage:SK6812MINI-E_fixed, F.Cu at (97.8, 55.5)
- added LED6: SK6812MINI-E, HackClubCarePackage:SK6812MINI-E_fixed, F.Cu at (118.6, 55.5)
- added LED7: SK6812MINI-E, HackClubCarePackage:SK6812MINI-E_fixed, F.Cu at (139.4, 55.5)
- added LED8: SK6812MINI-E, HackClubCarePackage:SK6812MINI-E_fixed, F.Cu at (160.2, 55.5)
- added LED9: SK6812MINI-E, HackClubCarePackage:SK6812MINI-E_fixed, F.Cu at (181.0, 55.5)
- added LED;1: SK6812MINI-E, HackClubCarePackage:SK6812MINI-E_fixed, F.Cu at (217.6, 97.1)
- added LED=1: SK6812MINI-E, HackClubCarePackage:SK6812MINI-E_fixed, F.Cu at (243.4, 55.5)
- added LEDA1: SK6812MINI-E, HackClubCarePackage:SK6812MINI-E_fixed, F.Cu at (30.4, 97.1)
- added LEDB1: SK6812MINI-E, HackClubCarePackage:SK6812MINI-E_fixed, F.Cu at (121.6, 117.9)
- added LEDBACK1: SK6812MINI-E, HackClubCarePackage:SK6812MINI-E_fixed, F.Cu at (273.6, 55.5)
- added LEDC1: SK6812MINI-E, HackClubCarePackage:SK6812MINI-E_fixed, F.Cu at (80.0, 117.9)
- added LEDCAPS1: SK6812MINI-E, HackClubCarePackage:SK6812MINI-E_fixed, F.Cu at (1.70, 97.1)
- added LEDD1: SK6812MINI-E, HackClubCarePackage:SK6812MINI-E_fixed, F.Cu at (72.0, 97.1)
- added LEDDEL1: SK6812MINI-E, HackClubCarePackage:SK6812MINI-E_fixed, F.Cu at (303.8, 55.5)
- added LEDDOWN1: SK6812MINI-E, HackClubCarePackage:SK6812MINI-E_fixed, F.Cu at (283.0, 138.7)
- added LEDE1: SK6812MINI-E, HackClubCarePackage:SK6812MINI-E_fixed, F.Cu at (66.6, 76.3)
- added LEDENTER1: SK6812MINI-E, HackClubCarePackage:SK6812MINI-E_fixed, F.Cu at (271.2, 97.1)
- added LEDESC1: SK6812MINI-E, HackClubCarePackage:SK6812MINI-E_fixed, F.Cu at (-6.20, 55.5)
- added LEDF1: SK6812MINI-E, HackClubCarePackage:SK6812MINI-E_fixed, F.Cu at (92.8, 97.1)
- added LEDG1: SK6812MINI-E, HackClubCarePackage:SK6812MINI-E_fixed, F.Cu at (113.6, 97.1)
- added LEDH1: SK6812MINI-E, HackClubCarePackage:SK6812MINI-E_fixed, F.Cu at (134.4, 97.1)
- added LEDI1: SK6812MINI-E, HackClubCarePackage:SK6812MINI-E_fixed, F.Cu at (170.6, 76.3)
- added LEDINS1: SK6812MINI-E, HackClubCarePackage:SK6812MINI-E_fixed, F.Cu at (303.8, 76.3)
- added LEDJ1: SK6812MINI-E, HackClubCarePackage:SK6812MINI-E_fixed, F.Cu at (155.2, 97.1)
- added LEDK1: SK6812MINI-E, HackClubCarePackage:SK6812MINI-E_fixed, F.Cu at (176.0, 97.1)
- added LEDL1: SK6812MINI-E, HackClubCarePackage:SK6812MINI-E_fixed, F.Cu at (196.8, 97.1)
- added LEDLALT1: SK6812MINI-E, HackClubCarePackage:SK6812MINI-E_fixed, F.Cu at (53.8, 138.7)
- added LEDLCTRL1: SK6812MINI-E, HackClubCarePackage:SK6812MINI-E_fixed, F.Cu at (-1.60, 138.7)
- added LEDLEFT1: SK6812MINI-E, HackClubCarePackage:SK6812MINI-E_fixed, F.Cu at (262.2, 138.7)
- added LEDLSHIFT1: SK6812MINI-E, HackClubCarePackage:SK6812MINI-E_fixed, F.Cu at (5.70, 117.9)
- added LEDLWIN1: SK6812MINI-E, HackClubCarePackage:SK6812MINI-E_fixed, F.Cu at (28.4, 138.7)
- added LEDM1: SK6812MINI-E, HackClubCarePackage:SK6812MINI-E_fixed, F.Cu at (163.2, 117.9)
- added LEDN1: SK6812MINI-E, HackClubCarePackage:SK6812MINI-E_fixed, F.Cu at (142.4, 117.9)
- added LEDO1: SK6812MINI-E, HackClubCarePackage:SK6812MINI-E_fixed, F.Cu at (191.4, 76.3)
- added LEDP1: SK6812MINI-E, HackClubCarePackage:SK6812MINI-E_fixed, F.Cu at (212.2, 76.3)
- added LEDPDN1: SK6812MINI-E, HackClubCarePackage:SK6812MINI-E_fixed, F.Cu at (303.8, 117.9)
- added LEDPUP1: SK6812MINI-E, HackClubCarePackage:SK6812MINI-E_fixed, F.Cu at (303.8, 97.1)
- added LEDQ1: SK6812MINI-E, HackClubCarePackage:SK6812MINI-E_fixed, F.Cu at (25.0, 76.3)
- added LEDR1: SK6812MINI-E, HackClubCarePackage:SK6812MINI-E_fixed, F.Cu at (87.4, 76.3)
- added LEDRALT1: SK6812MINI-E, HackClubCarePackage:SK6812MINI-E_fixed, F.Cu at (199.8, 138.7)
- added LEDRCTRL1: SK6812MINI-E, HackClubCarePackage:SK6812MINI-E_fixed, F.Cu at (241.4, 138.7)
- added LEDRIGHT1: SK6812MINI-E, HackClubCarePackage:SK6812MINI-E_fixed, F.Cu at (303.8, 138.7)
- added LEDRSHIFT1: SK6812MINI-E, HackClubCarePackage:SK6812MINI-E_fixed, F.Cu at (254.3, 117.9)
- added LEDRWIN1: SK6812MINI-E, HackClubCarePackage:SK6812MINI-E_fixed, F.Cu at (220.6, 138.7)
- added LEDS1: SK6812MINI-E, HackClubCarePackage:SK6812MINI-E_fixed, F.Cu at (51.2, 97.1)
- added LEDSPACE1: SK6812MINI-E, HackClubCarePackage:SK6812MINI-E_fixed, F.Cu at (129.0, 138.7)
- added LEDT1: SK6812MINI-E, HackClubCarePackage:SK6812MINI-E_fixed, F.Cu at (108.2, 76.3)
- added LEDTAB1: SK6812MINI-E, HackClubCarePackage:SK6812MINI-E_fixed, F.Cu at (-0.10, 76.3)
- added LEDU1: SK6812MINI-E, HackClubCarePackage:SK6812MINI-E_fixed, F.Cu at (149.8, 76.3)
- added LEDUP1: SK6812MINI-E, HackClubCarePackage:SK6812MINI-E_fixed, F.Cu at (283.0, 117.9)
- added LEDV1: SK6812MINI-E, HackClubCarePackage:SK6812MINI-E_fixed, F.Cu at (100.8, 117.9)
- added LEDW1: SK6812MINI-E, HackClubCarePackage:SK6812MINI-E_fixed, F.Cu at (45.8, 76.3)
- added LEDX1: SK6812MINI-E, HackClubCarePackage:SK6812MINI-E_fixed, F.Cu at (59.2, 117.9)
- added LEDY1: SK6812MINI-E, HackClubCarePackage:SK6812MINI-E_fixed, F.Cu at (129.0, 76.3)
- added LEDZ1: SK6812MINI-E, HackClubCarePackage:SK6812MINI-E_fixed, F.Cu at (38.4, 117.9)
- added LED[1: SK6812MINI-E, HackClubCarePackage:SK6812MINI-E_fixed, F.Cu at (233.0, 76.3)
- added LED\1: SK6812MINI-E, HackClubCarePackage:SK6812MINI-E_fixed, F.Cu at (278.8, 76.3)
- added LED]1: SK6812MINI-E, HackClubCarePackage:SK6812MINI-E_fixed, F.Cu at (253.8, 76.3)
- moved DDOWN1 13.2 mm to (293.3, 142.1)
- moved DENTER1 13.2 mm to (293.3, 100.5)
- moved DJ1 13.2 mm to (165.5, 100.5)
- moved DL1 13.2 mm to (207.1, 100.5)
- moved DPDN1 13.2 mm to (314.1, 121.3)
- moved DPUP1 13.2 mm to (314.1, 100.5)
- moved DRALT1 13.2 mm to (210.1, 142.1)
- moved DRCTRL1 13.2 mm to (251.7, 142.1)
- moved DRIGHT1 13.2 mm to (314.1, 142.1)
- moved DRWIN1 13.2 mm to (230.9, 142.1)
- moved STABSPACE1 13.2 mm to (129.0, 133.6)
- moved SWDOWN1 13.2 mm to (283.0, 133.6)
- moved SWLEFT1 13.2 mm to (262.2, 133.6)
- moved SWPDN1 13.2 mm to (303.8, 112.8)
- moved SWRIGHT1 13.2 mm to (303.8, 133.6)
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Connections:
- A2 pad 27: unconnected-(A2-GPIO21-Pad27) -> /Board LEDs/LEDs
Routing:
- net VCC: track 0.00 -> 1917.6 mm, vias 0 -> 12
- net Net-(LEDLALT1-DOUT): track 0.00 -> 70.6 mm
- net Net-(LEDRALT1-DIN): track 0.00 -> 66.2 mm
- net /Board LEDs/LEDs: track 0.00 -> 59.4 mm, vias 0 -> 2
- net Net-(LEDLCTRL1-DIN): track 0.00 -> 29.7 mm
- net Net-(LED'1-DOUT): track 0.00 -> 28.2 mm
- net Net-(LEDLSHIFT1-DIN): track 0.00 -> 28.1 mm, vias 0 -> 2
- net Net-(LEDENTER1-DOUT): track 0.00 -> 28.0 mm
- net Net-(LEDDEL1-DOUT): track 0.00 -> 26.5 mm
- net Net-(LEDCAPS1-DIN): track 0.00 -> 26.3 mm, vias 0 -> 2
- net Net-(LEDPDN1-DIN): track 0.00 -> 26.0 mm
- net Net-(LEDBACK1-DOUT): track 0.00 -> 25.6 mm
- net Net-(LED=1-DOUT): track 0.00 -> 25.6 mm
- net Net-(LEDLCTRL1-DOUT): track 0.00 -> 25.4 mm, vias 0 -> 2
- net Net-(LEDA1-DIN): track 0.00 -> 24.1 mm, vias 0 -> 2
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